File: power_usb.kicad_sch (KiCad schematic)
At the start: 12 parts, among them J5 USB_C_Receptacle_USB2.0_16P, J6 BAT, U8 AMS1117-3.3

Commit message: bom: fix using inconsistent value for same part
Parts:
- C18: value 100n -> 100nF
Changed lines of the file:
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@@
 			)
 		)
-		(property "Value" "100n"
+		(property "Value" "100nF"
 			(at 58.2168 131.953 0)
 			(effects

Commit message: schematic: Fixed LCSC part number for R45
Parts:
- R45: LCSC C4109 -> C25905
Changed lines of the file:
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@@
 			)
 		)
-		(property "LCSC" "C4109"
+		(property "LCSC" "C25905"
 			(at 48.26 49.53 90)
 			(effects
